File: kicad/Pico-DCO-1.sch (KiCad schematic (older format))
At the start: 21 parts, among them Q1 2N3904, U2 TL074

Commit message: Update silk screen
Parts:
- C3: value 1n -> 1n*
Other:
- note added: "* use polyester or similar"

Commit message: Add polyphony, update readme
Changed lines of the file:
@@
 AR Path="/60AE15A4/60873A52" Ref="R62"  Part="1"
 AR Path="/60AE2DA8/60873A52" Ref="R76"  Part="1"
-F 0 "R20" V 3693 2850 50  0000 C CNN
+F 0 "R76" V 3693 2850 50  0000 C CNN
 F 1 "100k" V 3784 2850 50  0000 C CNN
 F 2 "Resistor_THT:R_Axial_DIN0207_L6.3mm_D2.5mm_P10.16mm_Horizontal" V 3830 2850 50  0001 C CNN
@@
 AR Path="/60AE15A4/60873A58" Ref="R61"  Part="1"
 AR Path="/60AE2DA8/60873A58" Ref="R75"  Part="1"
-F 0 "R19" V 2893 3100 50  0000 C CNN
+F 0 "R75" V 2893 3100 50  0000 C CNN
 F 1 "100k" V 2984 3100 50  0000 C CNN
 F 2 "Resistor_THT:R_Axial_DIN0207_L6.3mm_D2.5mm_P10.16mm_Horizontal" V 3030 3100 50  0001 C CNN
@@
 AR Path="/60AE15A4/60873A7B" Ref="R71"  Part="1"
 AR Path="/60AE2DA8/60873A7B" Ref="R85"  Part="1"
-F 0 "R29" H 6280 4204 50  0000 R CNN
+F 0 "R85" H 6280 4204 50  0000 R CNN
 F 1 "100k" H 6280 4295 50  0000 R CNN
 F 2 "Resistor_THT:R_Axial_DIN0207_L6.3mm_D2.5mm_P10.16mm_Horizontal" V 6280 4250 50  0001 C CNN
@@
 AR Path="/60AE15A4/60873A81" Ref="C29"  Part="1"
 AR Path="/60AE2DA8/60873A81" Ref="C34"  Part="1"
-F 0 "C14" V 6355 3750 50  0000 C CNN
+F 0 "C34" V 6355 3750 50  0000 C CNN
 F 1 "10u" V 6264 3750 50  0000 C CNN
 F 2 "Capacitor_THT:CP_Radial_D5.0mm_P2.00mm" H 6138 3600 50  0001 C CNN
@@
 AR Path="/60AE15A4/60873A8A" Ref="U7"  Part="2"
 AR Path="/60AE2DA8/60873A8A" Ref="U8"  Part="2"
-F 0 "U4" H 3900 3567 50  0000 C CNN
+F 0 "U8" H 3900 3567 50  0000 C CNN
 F 1 "TL074" H 3900 3476 50  0000 C CNN
 F 2 "Package_DIP:DIP-14_W7.62mm_Socket_LongPads" H 3850 3300 50  0001 C CNN
@@
 AR Path="/60AE15A4/60873A9A" Ref="R64"  Part="1"
 AR Path="/60AE2DA8/60873A9A" Ref="R78"  Part="1"
-F 0 "R22" V 4343 3200 50  0000 C CNN
+F 0 "R78" V 4343 3200 50  0000 C CNN
 F 1 "100k" V 4434 3200 50  0000 C CNN
 F 2 "Resistor_THT:R_Axial_DIN0207_L6.3mm_D2.5mm_P10.16mm_Horizontal" V 4480 3200 50  0001 C CNN
@@
 AR Path="/60AE15A4/60873AA2" Ref="U7"  Part="1"
 AR Path="/60AE2DA8/60873AA2" Ref="U8"  Part="1"
-F 0 "U4" H 5300 3667 50  0000 C CNN
+F 0 "U8" H 5300 3667 50  0000 C CNN
 F 1 "TL074" H 5300 3576 50  0000 C CNN
 F 2 "Package_DIP:DIP-14_W7.62mm_Socket_LongPads" H 5250 3400 50  0001 C CNN
@@
 AR Path="/60AE15A4/60873ABA" Ref="C27"  Part="1"
 AR Path="/60AE2DA8/60873ABA" Ref="C32"  Part="1"
-F 0 "C12" V 3848 1550 50  0000 C CNN
+F 0 "C32" V 3848 1550 50  0000 C CNN
 F 1 "470p" V 3939 1550 50  0000 C CNN
 F 2 "Capacitor_THT:C_Rect_L7.2mm_W4.5mm_P5.00mm_FKS2_FKP2_MKS2_MKP2" H 4138 1400 50  0001 C CNN
@@
 AR Path="/60AE15A4/60873AC0" Ref="R63"  Part="1"
 AR Path="/60AE2DA8/60873AC0" Ref="R77"  Part="1"
-F 0 "R21" H 4520 1846 50  0000 L CNN
+F 0 "R77" H 4520 1846 50  0000 L CNN
 F 1 "10k" H 4520 1755 50  0000 L CNN
 F 2 "Resistor_THT:R_Axial_DIN0207_L6.3mm_D2.5mm_P10.16mm_Horizontal" V 4380 1800 50  0001 C CNN
@@
 AR Path="/60AE15A4/60873AC6" Ref="R65"  Part="1"
 AR Path="/60AE2DA8/60873AC6" Ref="R79"  Part="1"
-F 0 "R23" V 4593 1550 50  0000 C CNN
+F 0 "R79" V 4593 1550 50  0000 C CNN
 F 1 "1k" V 4684 1550 50  0000 C CNN
 F 2 "Resistor_THT:R_Axial_DIN0207_L6.3mm_D2.5mm_P10.16mm_Horizontal" V 4730 1550 50  0001 C CNN
@@
 AR Path="/60AE15A4/60873ACC" Ref="R69"  Part="1"
 AR Path="/60AE2DA8/60873ACC" Ref="R83"  Part="1"
-F 0 "R27" H 5720 2396 50  0000 L CNN
+F 0 "R83" H 5720 2396 50  0000 L CNN
 F 1 "2k2" H 5720 2305 50  0000 L CNN
 F 2 "Resistor_THT:R_Axial_DIN0207_L6.3mm_D2.5mm_P10.16mm_Horizontal" V 5580 2350 50  0001 C CNN
@@
 AR Path="/60AE15A4/60873AD2" Ref="C28"  Part="1"
 AR Path="/60AE2DA8/60873AD2" Ref="C33"  Part="1"
-F 0 "C13" V 5048 2700 50  0000 C CNN
+F 0 "C33" V 5048 2700 50  0000 C CNN
 F 1 "1n*" V 5139 2700 50  0000 C CNN
 F 2 "Capacitor_THT:C_Rect_L7.2mm_W4.5mm_P5.00mm_FKS2_FKP2_MKS2_MKP2" H 5338 2550 50  0001 C CNN
@@
 AR Path="/60AE15A4/60873AD8" Ref="Q5"  Part="1"
 AR Path="/60AE2DA8/60873AD8" Ref="Q6"  Part="1"
-F 0 "Q2" V 5535 1900 50  0000 C CNN
+F 0 "Q6" V 5535 1900 50  0000 C CNN
 F 1 "2N3904" V 5626 1900 50  0000 C CNN
 F 2 "Package_TO_SOT_THT:TO-92_Wide" H 5500 1825 50  0001 L CIN
@@
 AR Path="/60AE15A4/60873ADE" Ref="U7"  Part="4"
 AR Path="/60AE2DA8/60873ADE" Ref="U8"  Part="4"
-F 0 "U4" H 6200 5867 50  0000 C CNN
+F 0 "U8" H 6200 5867 50  0000 C CNN
 F 1 "TL074" H 6200 5776 50  0000 C CNN
 F 2 "Package_DIP:DIP-14_W7.62mm_Socket_LongPads" H 6150 5600 50  0001 C CNN
@@
 AR Path="/60AE15A4/60873AE5" Ref="R70"  Part="1"
 AR Path="/60AE2DA8/60873AE5" Ref="R84"  Part="1"
-F 0 "R28" H 5580 4204 50  0000 R CNN
+F 0 "R84" H 5580 4204 50  0000 R CNN
 F 1 "10k" H 5580 4295 50  0000 R CNN
 F 2 "Resistor_THT:R_Axial_DIN0207_L6.3mm_D2.5mm_P10.16mm_Horizontal" V 5580 4250 50  0001 C CNN
@@
 AR Path="/60AE15A4/60873AF2" Ref="R68"  Part="1"
 AR Path="/60AE2DA8/60873AF2" Ref="R82"  Part="1"
-F 0 "R26" H 5370 5996 50  0000 L CNN
+F 0 "R82" H 5370 5996 50  0000 L CNN
 F 1 "470k" H 5370 5905 50  0000 L CNN
 F 2 "Resistor_THT:R_Axial_DIN0207_L6.3mm_D2.5mm_P10.16mm_Horizontal" V 5230 5950 50  0001 C CNN
@@
 AR Path="/60AE15A4/60873AF8" Ref="R66"  Part="1"
 AR Path="/60AE2DA8/60873AF8" Ref="R80"  Part="1"
-F 0 "R24" V 5007 4650 50  0000 C CNN
+F 0 "R80" V 5007 4650 50  0000 C CNN
 F 1 "150k" V 4916 4650 50  0000 C CNN
 F 2 "Resistor_THT:R_Axial_DIN0207_L6.3mm_D2.5mm_P10.16mm_Horizontal" V 4730 4650 50  0001 C CNN
@@
 AR Path="/60AE15A4/60873AFE" Ref="R67"  Part="1"
 AR Path="/60AE2DA8/60873AFE" Ref="R81"  Part="1"
-F 0 "R25" V 5007 5600 50  0000 C CNN
+F 0 "R81" V 5007 5600 50  0000 C CNN
 F 1 "100k" V 4916 5600 50  0000 C CNN
 F 2 "Resistor_THT:R_Axial_DIN0207_L6.3mm_D2.5mm_P10.16mm_Horizontal" V 4730 5600 50  0001 C CNN
@@
 AR Path="/60AE15A4/60873B1E" Ref="R72"  Part="1"
 AR Path="/60AE2DA8/60873B1E" Ref="R86"  Part="1"
-F 0 "R30" V 6593 5500 50  0000 C CNN
+F 0 "R86" V 6593 5500 50  0000 C CNN
 F 1 "10k" V 6684 5500 50  0000 C CNN
 F 2 "Resistor_THT:R_Axial_DIN0207_L6.3mm_D2.5mm_P10.16mm_Horizontal" V 6730 5500 50  0001 C CNN
@@
 AR Path="/60AE15A4/60873B24" Ref="R73"  Part="1"
 AR Path="/60AE2DA8/60873B24" Ref="R87"  Part="1"
-F 0 "R31" H 7120 5796 50  0000 L CNN
+F 0 "R87" H 7120 5796 50  0000 L CNN
 F 1 "5k6" H 7120 5705 50  0000 L CNN
 F 2 "Resistor_THT:R_Axial_DIN0207_L6.3mm_D2.5mm_P10.16mm_Horizontal" V 6980 5750 50  0001 C CNN
@@
 AR Path="/60AE15A4/60873B5B" Ref="R60"  Part="1"
 AR Path="/60AE2DA8/60873B5B" Ref="R74"  Part="1"
-F 0 "R18" V 2293 3100 50  0000 C CNN
+F 0 "R74" V 2293 3100 50  0000 C CNN
 F 1 "4k7" V 2384 3100 50  0000 C CNN
 F 2 "Resistor_THT:R_Axial_DIN0207_L6.3mm_D2.5mm_P10.16mm_Horizontal" V 2430 3100 50  0001 C CNN
@@
 AR Path="/60AE15A4/60873B69" Ref="C26"  Part="1"
 AR Path="/60AE2DA8/60873B69" Ref="C31"  Part="1"
-F 0 "C11" V 2548 3400 50  0000 C CNN
+F 0 "C31" V 2548 3400 50  0000 C CNN
 F 1 "100n" V 2639 3400 50  0000 C CNN
 F 2 "Capacitor_THT:C_Rect_L7.2mm_W4.5mm_P5.00mm_FKS2_FKP2_MKS2_MKP2" H 2838 3250 50  0001 C CNN
@@
 AR Path="/60AE15A4/60873A65" Ref="U7"  Part="3"
 AR Path="/60AE2DA8/60873A65" Ref="U8"  Part="3"
-F 0 "U4" H 7350 4217 50  0000 C CNN
+F 0 "U8" H 7350 4217 50  0000 C CNN
 F 1 "TL074" H 7350 4126 50  0000 C CNN
 F 2 "Package_DIP:DIP-14_W7.62mm_Socket_LongPads" H 7300 3950 50  0001 C CNN
@@
 AR Path="/60AE15A4/60926AFD" Ref="U7"  Part="5"
 AR Path="/60AE2DA8/60926AFD" Ref="U8"  Part="5"
-F 0 "U4" H 9958 5596 50  0000 L CNN
+F 0 "U8" H 9958 5596 50  0000 L CNN
 F 1 "TL074" H 9958 5505 50  0000 L CNN
 F 2 "" H 9950 5650 50  0001 C CNN
@@
 AR Path="/60AE15A4/609307F0" Ref="C30"  Part="1"
 AR Path="/60AE2DA8/609307F0" Ref="C35"  Part="1"
-F 0 "C15" V 9398 5600 50  0000 C CNN
+F 0 "C35" V 9398 5600 50  0000 C CNN
 F 1 "100n" V 9489 5600 50  0000 C CNN
 F 2 "Capacitor_THT:C_Rect_L7.2mm_W4.5mm_P5.00mm_FKS2_FKP2_MKS2_MKP2" H 9688 5450 50  0001 C CNN
